File: Board/io2.kicad_sch (KiCad schematic)
At the start: 9 parts, among them P2 IEEE488FLATCABLE, U1 XC6SLX9-TQG144, U4 SN75160BDW, U5 SN75161BDW, U6 LSF0204Q, U7 LSF0204Q, U8 LSF0204Q, U9 LSF0204Q

Commit message: update
Connections:
- net V33: now reaches U1.103 (VCCO_1)
- net V33: now also U1.122 (VCCO_0), U1.125 (VCCO_0), U1.135 (VCCO_0), U1.76 (VCCO_1), U1.86 (VCCO_1)
Other:
- moved on the sheet: P2, R3, U1A, U4, U5, U6, U7, U8, U9

Commit message: adding keyboard, serial IEC
Parts:
- added C1: 100n, Capacitor_SMD:C_0805_2012Metric, symbol Device:C
- added J1: DIN-6, csa_petio_v1:DIN6PIEC, symbol Connector:DIN-6
- added J14: Extended_PET_keyboard_connector, csa_petio_v1:PET_Extended_Keyboard_Connector, symbol petkn:Extended_PET_keyboard_connector
- added J2: Conn_01x23, Connector_PinSocket_2.54mm:PinSocket_1x23_P2.54mm_Vertical, symbol Connector_Generic:Conn_01x23
- added JP18, JP22: JP1E, Connector_PinHeader_2.54mm:PinHeader_1x02_P2.54mm_Vertical, symbol cbm_ultipet_v1-eagle-import:JP1E
- added RN1: 10k, Resistor_THT:R_Array_SIP9, symbol Device:R_Network08
- added U10: 74LS06, Package_SO:SO-14_3.9x8.65mm_P1.27mm, symbol 74xx:74LS06
- added U11: SN74LVC245APW, Package_SO:TSSOP-20_4.4x6.5mm_P0.65mm, symbol Logic_LevelTranslator:SN74LVC245APW
- added U12, U13: 4051, Package_SO:SOP-16_3.9x9.9mm_P1.27mm, symbol 4xxx:4051
- added U14: 74LVC1G04, Package_TO_SOT_SMD:SOT-23-5, symbol 74xGxx:74LVC1G04
Connections:
- net V33 is gone; now on net VCC: U1.103 (VCCO_1), U1.122 (VCCO_0), U1.125 (VCCO_0), U1.135 (VCCO_0), U1.76 (VCCO_1), U1.86 (VCCO_1)
- net GND: now also C1.2, J1.2, J14.1, J14.21 (GND), U10.7 (GND), U11.10 (GND), U12.3 (X), U12.7 (VEE), U12.8 (VSS), U13.3 (X), U13.7 (VEE), U13.8 (VSS), U14.3 (GND)
- net VCC: now also C1.1, J14.26 (VCC5), J14.27 (VCC33), RN1.1 (common), U10.14 (VCC), U11.1 (DIR), U11.20 (VCC), U12.16 (VDD), U13.16 (VDD), U14.5 (VCC)
- net /RES: now also JP22.2
- net at U1.114 (IO_L65N_SCP2_0): now also J14.13, RN1.2 (R1)
- net at U1.115 (IO_L65P_SCP3_0): now also J14.14, RN1.3 (R2)
- net at U1.116 (IO_L64N_SCP4_0): now also J14.15, J2.1 (Pin_1), RN1.4 (R3)
- net at U1.117 (IO_L64P_SCP5_0): now also J14.16, J2.2 (Pin_2), RN1.5 (R4)
- net at U1.118 (IO_L63N_SCP6_0): now also J14.17, J2.3 (Pin_3), RN1.6 (R5)
- net at U1.119 (IO_L63P_SCP7_0): now also J14.18, J2.4 (Pin_4), RN1.7 (R6)
- net at U1.120 (IO_L62N_VREF_0): now also J14.19, J2.5 (Pin_5), RN1.8 (R7)
- net at U1.121 (IO_L62P_0): now also J14.20, J2.6 (Pin_6), RN1.9 (R8)
- net KSEL0: now reaches U1.123 (IO_L37N_GCLK12_0)
- net KSEL0: now also J14.22 (S0), U12.11 (A), U13.11 (A)
- net KSEL1: now reaches U1.124 (IO_L37P_GCLK13_0)
- net KSEL1: now also J14.23 (S1), U12.10 (B), U13.10 (B)
- net KSEL2: now reaches U1.126 (IO_L36N_GCLK14_0)
- net KSEL2: now also J14.24 (S2), U12.9 (C), U13.9 (C)
- net KSEL3: now reaches U1.127 (IO_L36P_GCLK15_0)
- net KSEL3: now also J14.25 (S3), U12.6 (Inh), U14.2
- net at U1.131 (IO_L35N_GCLK16_0): now also U10.1
- net at U1.132 (IO_L35P_GCLK17_0): now also U10.3
- net at U1.133 (IO_L34N_GCLK18_0): now also U10.5
- net at U1.134 (IO_L34P_GCLK19_0): now also U10.9
- net at U1.137 (IO_L4N_0): now also U11.11 (B8)
- net at U1.138 (IO_L4P_0): now also U11.12 (B7)
- net at U1.139 (IO_L3N_0): now also U11.13 (B6)
- net at U1.140 (IO_L3P_0): now also U11.14 (B5)
- net at U1.141 (IO_L2N_0): now also U11.15 (B4)
- net at U1.142 (IO_L2P_0): now also U11.16 (B3)
- net at U1.143 (IO_L1N_VREF_0): now also U11.17 (B2)
- net at U1.144 (IO_L1P_HSWAPEN_0): now also U11.18 (B1)
- new net: J2.10 (Pin_10), U13.1 (X4)
- new net: J2.11 (Pin_11), U13.12 (X3)
- new net: J14.4, J2.14 (Pin_14), U13.13 (X0)
- new net: J14.3, J2.13 (Pin_13), U13.14 (X1)
- new net: J14.2, J2.12 (Pin_12), U13.15 (X2)
- new net: J2.8 (Pin_8), U13.2 (X6)
- new net: J2.7 (Pin_7), U13.4 (X7)
- new net: J2.9 (Pin_9), U13.5 (X5)
- new net: U13.6 (Inh), U14.4
- new net: J14.5, J2.15 (Pin_15), U12.4 (X7)
- new net: J14.6, J2.16 (Pin_16), U12.2 (X6)
- new net: J14.7, J2.17 (Pin_17), U12.5 (X5)
- new net: J14.8, J2.18 (Pin_18), U12.1 (X4)
- new net: J14.9, J2.19 (Pin_19), U12.12 (X3)
- new net: J14.10, J2.20 (Pin_20), U12.15 (X2)
- new net: J14.11, J2.21 (Pin_21), JP22.1, U12.14 (X1)
- new net: J14.12, J2.23 (Pin_23), JP18.1, U12.13 (X0)
- new net: J1.3, U10.2, U11.2 (A1)
- new net: J1.1, U10.4, U11.5 (A4)
- new net: J1.5, U10.6, U11.3 (A2)
- new net: J1.4, U10.8, U11.4 (A3)
- new net SCL: J14.28 (SCL)
- new net SDA: J14.29 (SCA)
- new net /IRQ: JP18.2
Other:
- note added: "For use with two-row IDC keyboard connector"
- moved on the sheet: P2, R3, U1A, U4, U5, U6, U7, U8, U9

Commit message: add serial, SPI-10-5V
Connections:
- net SATN: now reaches J1.3, U10.2, U11.2 (A1)
- net FASTCLK: now reaches J1.1, U10.4, U11.5 (A4)
- net DATA: now reaches J1.5, U10.6, U11.3 (A2)
- net SLOWCLK: now reaches J1.4, U10.8, U11.4 (A3)
- net CLKOUT: now reaches U1.134 (IO_L34P_GCLK19_0), U10.9
Other:
- note added: "CSA-CBMIO-V1.0A"
- note removed: "CSA-PETIO-V1.3B"
- moved on the sheet: U1A

Commit message: schematics 1st full rev
Parts:
- removed C1: 100n, Capacitor_SMD:C_0805_2012Metric, symbol Device:C
- added R10, R9: 1k, Resistor_SMD:R_0603_1608Metric_Pad0.98x0.95mm_HandSolder, symbol Device:R
- added RN2, RN3: 10k, Resistor_THT:R_Array_SIP9, symbol Device:R_Network08
Connections:
- net CLKOUT: now also U1.144 (IO_L1P_HSWAPEN_0); no longer U1.134 (IO_L34P_GCLK19_0)
- net GND: now also R10.2, R9.2
- net VCC: now also U6.1 (VRefA), U6.14 (VRefB), U7.1 (VRefA), U7.14 (VRefB), U8.1 (VRefA), U8.14 (VRefB), U9.1 (VRefA), U9.14 (VRefB), RN2.1 (common), RN3.1 (common)
- net at U4.1 (TE), U5.1 (TE): now also U1.83 (IO_L45P_1); no longer U1.84 (IO_L43N_GCLK4_1)
- net at U5.11 (DC): now also U1.82 (IO_L45N_1); no longer U1.83 (IO_L45P_1)
- net at U5.12 (SRQ), U9.10 (B4): now also RN3.2 (R1)
- net at U5.13 (ATN), U9.11 (B3): now also RN3.3 (R2)
- net at U5.14 (EOI), U9.12 (B2): now also RN3.4 (R3)
- net at U5.15 (DAV), U9.13 (B1): now also RN3.5 (R4)
- net at U5.16 (NRFD), U8.10 (B4): now also RN3.6 (R5)
- net at U5.17 (NDAC), U8.11 (B3): now also RN3.7 (R6)
- net at U5.18 (IFC), U8.12 (B2): now also RN3.8 (R7)
- net at U5.19 (REN), U8.13 (B1): now also RN3.9 (R8)
- net at U11.11 (B8): no longer U1.137 (IO_L4N_0)
- net at U11.12 (B7): no longer U1.138 (IO_L4P_0)
- net at U11.13 (B6): no longer U1.139 (IO_L3N_0)
- net at U11.14 (B5): no longer U1.140 (IO_L3P_0)
- net at U11.18 (B1): now also U1.134 (IO_L34P_GCLK19_0); no longer U1.144 (IO_L1P_HSWAPEN_0)
- net at U11.6 (A5): now also U11.7 (A6), U11.8 (A7), U11.9 (A8), R9.1
- net UD4: now reaches U4.16 (D4), U6.10 (B4)
- net UD4: now also RN2.5 (R4)
- net UD3: now reaches U4.17 (D3), U6.11 (B3)
- net UD3: now also RN2.4 (R3)
- net UD2: now reaches U4.18 (D2), U6.12 (B2)
- net UD2: now also RN2.3 (R2)
- net UD1: now reaches U4.19 (D1), U6.13 (B1)
- net UD1: now also RN2.2 (R1)
- net at U6.2 (A1): now also U1.105 (IO_L1P_1)
- net at U6.3 (A2): now also U1.104 (IO_L1N_VREF_1); no longer U1.105 (IO_L1P_1)
- net at U6.4 (A3): now also U1.102 (IO_L32P_1); no longer U1.104 (IO_L1N_VREF_1)
- net at U6.5 (A4): now also U1.101 (IO_L32N_1); no longer U1.102 (IO_L32P_1)
- net at U1.100 (IO_L33P_1): now also U7.2 (A1); no longer U7.3 (A2)
- net UP7: now reaches U1.111 (IO_L66N_SCP0_0)
- net UP6: now reaches U1.112 (IO_L66P_SCP1_0)
- net UP5: now reaches U1.74 (IO_L74N_DOUT_BUSY_1)
- net UP4: now reaches U1.75 (IO_L74P_AWAKE_1)
- net UP3: now reaches U1.78 (IO_L47N_1)
- net UP2: now reaches U1.79 (IO_L47P_1)
- net UP1: now reaches U1.80 (IO_L46N_1)
- net UP0: now reaches U1.81 (IO_L46P_1)
- net at U9.5 (A4): now also U1.84 (IO_L43N_GCLK4_1); no longer U1.85 (IO_L43P_GCLK5_1)
- net at U9.4 (A3): now also U1.85 (IO_L43P_GCLK5_1); no longer U1.87 (IO_L42N_GCLK6_TRDY1_1)
- net at U9.3 (A2): now also U1.87 (IO_L42N_GCLK6_TRDY1_1); no longer U1.88 (IO_L42P_GCLK7_1)
- net at U9.2 (A1): now also U1.88 (IO_L42P_GCLK7_1); no longer U1.92 (IO_L41N_GCLK8_1)
- net at U8.5 (A4): now also U1.92 (IO_L41N_GCLK8_1); no longer U1.93 (IO_L41P_GCLK9_IRDY1_1)
- net at U8.4 (A3): now also U1.93 (IO_L41P_GCLK9_IRDY1_1); no longer U1.94 (IO_L40N_GCLK10_1)
- net at U8.3 (A2): now also U1.94 (IO_L40N_GCLK10_1); no longer U1.95 (IO_L40P_GCLK11_1)
- net at U8.2 (A1): now also U1.95 (IO_L40P_GCLK11_1); no longer U1.97 (IO_L34N_1)
- net at U7.5 (A4): now also U1.97 (IO_L34N_1); no longer U1.98 (IO_L34P_1)
- net at U7.4 (A3): now also U1.98 (IO_L34P_1); no longer U1.99 (IO_L33N_1)
- net UD8: now reaches U4.12 (D8), U7.10 (B4)
- net UD8: now also RN2.9 (R8)
- net UD7: now reaches U4.13 (D7), U7.11 (B3)
- net UD7: now also RN2.8 (R7)
- net UD6: now reaches U4.14 (D6), U7.12 (B2)
- net UD6: now also RN2.7 (R6)
- net UD5: now reaches U4.15 (D5), U7.13 (B1)
- net UD5: now also RN2.6 (R5)
- net at U10.11: now also R10.1
- new net: U1.99 (IO_L33N_1), U7.3 (A2)
- new net UP10: U1.138 (IO_L4P_0)
- new net UP11: U1.137 (IO_L4N_0)
- new net UP8: U1.140 (IO_L3P_0)
- new net UP9: U1.139 (IO_L3N_0)
Other:
- note added: "CSA-CBMIO-V1.0A-20250815"
- note added: "Note: - FPGA has do to internal pull-ups - 7516x are LS type which should have internal pull-ups. Optional external pull ups can be used"
- note removed: "CSA-PETIO-V1.3B-20240214"
- moved on the sheet: P2, R3, U4, U5, U6

Commit message: full connect, starting on prod
Parts:
- added RN6: 4k7, Resistor_THT:R_Array_SIP5, symbol Device:R_Network04
- P2: footprint csa_petio_v1:FLAT24 -> csa_petio_v1:FLAT24_IDC
Connections:
- net DATA: now also RN6.4 (R3)
- net FASTCLK: now also RN6.3 (R2)
- net SATN: now also RN6.2 (R1)
- net SLOWCLK: now also RN6.5 (R4)
- net VCC: now also RN6.1 (common); no longer J14.27 (VCC33), RN1.1 (common), U1.103 (VCCO_1), U1.122 (VCCO_0), U1.125 (VCCO_0), U1.135 (VCCO_0), U1.76 (VCCO_1), U1.86 (VCCO_1), U11.1 (DIR), U11.20 (VCC), U12.16 (VDD), U13.16 (VDD), U14.5 (VCC), U6.1 (VRefA), U7.1 (VRefA), U8.1 (VRefA), U9.1 (VRefA)
- new net V33: J14.27 (VCC33), RN1.1 (common), U1.103 (VCCO_1), U1.122 (VCCO_0), U1.125 (VCCO_0), U1.135 (VCCO_0), U1.76 (VCCO_1), U1.86 (VCCO_1), U11.1 (DIR), U11.20 (VCC), U12.16 (VDD), U13.16 (VDD), U14.5 (VCC), U6.1 (VRefA), U7.1 (VRefA), U8.1 (VRefA), U9.1 (VRefA)
