File: Board/io2.kicad_sch (KiCad schematic)
At the start: 25 parts, among them J1 DIN-6, J14 Extended_PET_keyboard_connect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, J2 Conn_01x23, P2 IEEE488FLATCABLE, U1 XC6SLX9-TQG144, U10 74LS06, U11 SN74LVC245APW, U12 4051, U13 4051, U14 74LVC1G04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

Commit message: 1st working as 1.0B
Other:
- note added: "CSA-CBMIO-V1.0B"
- note removed: "CSA-CBMIO-V1.0A"
Changed lines of the file:
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@@
 		)
 	)
-	(text "CSA-CBMIO-V1.0A"
+	(text "CSA-CBMIO-V1.0B"
 		(exclude_from_sim no)
 		(at 339.09 261.112 0)
