File: Board/io2.kicad_sch (KiCad schematic)
At the start: 25 parts, among them J1 DIN-6, J14 Extended_PET_keyboard_connect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, J2 Conn_01x23, P2 IEEE488FLATCABLE, U1 XC6SLX9-TQG144, U10 74LS06, U11 SN74LVC245APW, U12 4051, U13 4051, U14 74LVC1G04, U4 SN75160BDW, U5 SN75161BDW, U6 LSF0204Q, U7 LSF0204Q, U8 LSF0204Q, U9 LSF0204Q

Commit message: add par ATNA, separate kbd cons, kbd serial input to get more I/O
Parts:
- removed J14: Extended_PET_keyboard_connector, csa_petio_v1:PET_Extended_Keyboard_Connector, symbol petkn:Extended_PET_keyboard_connector
- removed JP18, JP22: JP1E, Connector_PinHeader_2.54mm:PinHeader_1x02_P2.54mm_Vertical, symbol cbm_ultipet_v1-eagle-import:JP1E
- removed R10: 1k, Resistor_SMD:R_0603_1608Metric_Pad0.98x0.95mm_HandSolder, symbol Device:R
- removed U14: 74LVC1G04, Package_TO_SOT_SMD:SOT-23-5, symbol 74xGxx:74LVC1G04
- added C171: 51pF, cbm_ultipet_v1:C025-024X044, symbol cbm_ultipet_v1-eagle-import:C-EU025-024X044
- added C172: 360p, cbm_ultipet_v1:C025-024X044, symbol cbm_ultipet_v1-eagle-import:C-EU025-024X044
- added J3: New_PET_keyboard_connector, Connector_IDC:IDC-Header_2x10_P2.54mm_Vertical, symbol petkn:New_PET_keyboard_connector
- added P8: (no value), Connector_PinHeader_2.54mm:PinHeader_1x20_P2.54mm_Vertical, symbol cbm_ultipet_v1-eagle-import:PETKEYBD
- added Q4: BC557, cbm_ultipet_v1:TO92, symbol cbm_ultipet_v1-eagle-import:BC557
- added R47, R48: 10k, Resistor_SMD:R_0805_2012Metric_Pad1.20x1.40mm_HandSolder, symbol csa_ultracpu-eagle-import:R-EU_0207/2V
- added R68, R69: 1M, cbm_ultipet_v1:0207_2V, symbol cbm_ultipet_v1-eagle-import:R-EU_0207/2V
- added R70: 47k, cbm_ultipet_v1:0207_2V, symbol cbm_ultipet_v1-eagle-import:R-EU_0207/2V
- added R71: 100k, cbm_ultipet_v1:0207_7, symbol cbm_ultipet_v1-eagle-import:R-EU_0207/7
- added U14: 74LVC2G06, symbol 74xGxx:74LVC2G06
- added U24: 74LVC165, Package_SO:TSSOP-16_4.4x5mm_P0.65mm, symbol 74xx:74LS165
- added U25: NE555D, Package_SO:SOIC-8_3.9x4.9mm_P1.27mm, symbol Timer:NE555D
- added X1: 18.432MHz, Oscillator:Oscillator_SMD_SeikoEpson_SG8002CE-4Pin_3.2x2.5mm, symbol Oscillator:SG-8002CE
Connections:
- net GND: now also C172.1, J3.19 (GND), P8.1 (GND), Q4.3 (C), U14.2 (GND), U24.10 (DS), U24.15 (~{CE}), U24.8 (GND), U25.1 (GND), X1.2 (GND)
- net KSEL0: now also J3.17 (S0)
- net KSEL1: now also J3.15 (S1)
- net KSEL2: now also J3.13 (S2)
- net KSEL3: now also U10.11, J3.11 (S3)
- net NDAC: now also U14.6
- net NRFD: now also U14.4
- net SCL: now also J3.5 (SCL)
- net SDA: now also J3.3 (SCA)
- net V33: now also J3.7 (VCC33), R47.1, R48.1, R68.1, U14.5 (VCC), U24.16 (VCC), X1.4 (Vcc)
- net VCC: now also J3.9 (VCC5), R69.1, R70.2, U25.4 (R), U25.8 (VCC)
- net /IRQ: now also J3.2 (/IRQ)
- net /RES: now also J3.4 (/RES)
- net at J2.14 (Pin_14), U13.13 (X0): now also P8.4 (DEC8)
- net at J2.13 (Pin_13), U13.14 (X1): now also P8.3 (DEC9)
- net at U13.6 (Inh): now also U10.10, R48.2
- net at J2.1 (Pin_1), RN1.4 (R3): now also J3.10 (C6), P8.15 (KIN5), U24.4 (D5); no longer U1.116 (IO_L64N_SCP4_0)
- net at J2.15 (Pin_15), U12.4 (X7): now also P8.5 (DEC7)
- net at J2.16 (Pin_16), U12.2 (X6): now also P8.6 (DEC6)
- net at J2.17 (Pin_17), U12.5 (X5): now also P8.7 (DEC5)
- net at J2.18 (Pin_18), U12.1 (X4): now also P8.8 (DEC4)
- net at J2.19 (Pin_19), U12.12 (X3): now also P8.9 (DEC3)
- net at J2.2 (Pin_2), RN1.5 (R4): now also J3.12 (C5), P8.16 (KIN4), U24.3 (D4); no longer U1.117 (IO_L64P_SCP5_0)
- net at J2.20 (Pin_20), U12.15 (X2): now also P8.10 (DEC2)
- net at J2.21 (Pin_21), U12.14 (X1): now also P8.11 (DEC1)
- net at J2.23 (Pin_23), U12.13 (X0): now also P8.12 (DEC0)
- net at J2.3 (Pin_3), RN1.6 (R5): now also J3.14 (C4), P8.17 (KIN3), U24.14 (D3); no longer U1.118 (IO_L63N_SCP6_0)
- net at J2.4 (Pin_4), RN1.7 (R6): now also J3.16 (C3), P8.18 (KIN2), U24.13 (D2); no longer U1.119 (IO_L63P_SCP7_0)
- net at J2.5 (Pin_5), RN1.8 (R7): now also J3.18 (C2), P8.19 (KIN1), U24.12 (D1); no longer U1.120 (IO_L62N_VREF_0)
- net at J2.6 (Pin_6), RN1.9 (R8): now also J3.20 (C1), P8.20 (KIN0), U24.11 (D0); no longer U1.121 (IO_L62P_0)
- net at RN1.2 (R1): now also J3.6 (C8), P8.13 (KIN7), U24.6 (D7); no longer U1.114 (IO_L65N_SCP2_0)
- net at RN1.3 (R2): now also J3.8 (C7), P8.14 (KIN6), U24.5 (D6); no longer U1.115 (IO_L65P_SCP3_0)
- new net: Q4.2 (B), R71.1
- new net: R71.2, U25.3 (Q)
- new net: U1.117 (IO_L64P_SCP5_0), U14.1, U14.3
- new net: C171.1, J3.1 (RESTORE), R68.2
- new net: C171.2, R69.2, U25.2 (TR)
- new net: R47.2, X1.1 (OE)
- new net: U1.118 (IO_L63N_SCP6_0), X1.3 (OUT)
- new net: U1.119 (IO_L63P_SCP7_0), U24.9 (Q7)
- new net: U1.120 (IO_L62N_VREF_0), U24.1 (~{PL})
- new net: U1.121 (IO_L62P_0), U24.2 (CP)
- new net: C172.2, R70.1, U25.6 (THR), U25.7 (DIS)
- new net /BNMI: Q4.1 (E)
Other:
- note added: "CSA-CBMIO-V1.1A"
- note added: "Note: - FPGA has do to internal pull-ups"
- note added: "RESTORE to NMI from C64"
- note removed: "CSA-CBMIO-V1.0B"
- note removed: "For use with two-row IDC keyboard connector"
- note removed: "Note: - FPGA has do to internal pull-ups - Par ATNA handling is still missing, need one more I/O pins for Parallel ATNA. Serial can be done inside the FPGA"
- moved on the sheet: J2, RN1, U10E, U12, U13

Commit message: schem draft done, layout work started
Parts:
- removed Q4: BC557, cbm_ultipet_v1:TO92, symbol cbm_ultipet_v1-eagle-import:BC557
- removed R71: 100k, cbm_ultipet_v1:0207_7, symbol cbm_ultipet_v1-eagle-import:R-EU_0207/7
- removed U14: 74LVC2G06, symbol 74xGxx:74LVC2G06
- added U14: 74LS06, Package_SO:SO-14_3.9x8.65mm_P1.27mm, symbol 74xx:74LS06
- C171, C172: footprint cbm_ultipet_v1:C025-024X044 -> Capacitor_SMD:C_0805_2012Metric
- R3, R9: value 1k -> 4k7
- R47, R48: value 10k -> 4k7
- R68, R69, R70: footprint cbm_ultipet_v1:0207_2V -> Resistor_SMD:R_0603_1608Metric_Pad0.98x0.95mm_HandSolder
Connections:
- net GND: now also U14.7 (GND)
- net NDAC: now also U14.2
- net NRFD: now also U14.4
- net VCC: now also U14.14 (VCC)
- net /BNMI: now also U14.6
- net at U25.3 (Q): now also U14.5
- net at U1.117 (IO_L64P_SCP5_0): now also U14.1, U14.3
- net UP14: now reaches U1.116 (IO_L64N_SCP4_0)
Other:
- note added: "CSA-CBMIO-V1.1A-20260824"
- note added: "V1.1A: - Adding a 74LVC165 to clock in keyboard input instead of 8 parallel gives 5 more free I/O for Par ATNA, joy setup, ... - separate connectors for PET and UPET keyboards - UPET kbd -> restore key to NMI - Replace U14 with U10E + pullup - Parallel ATNA handling"
- note removed: "CSA-CBMIO-V1.0A-20250815"
- note removed: "TODO: - Adding a 74LVC165 to clock in keyboard input instead of 8 parallel gives 5 more free I/O for Par ATNA, joy setup, ... - separate connectors for PET and UPET keyboards - UPET kbd (now pin 30) -> restore key to NMI - Replace U14 with U10E + pullup"
- moved on the sheet: J2, R48, RN1, U10E, U12, U13, U24

Commit message: more layout work
Parts:
- added unit 2 of U14
- added unit 3 of U14
- added unit 1 of U14
Connections:
- net NDAC: now also U14.2; no longer U14.2
- net NRFD: now also U14.4; no longer U14.4
- net /BNMI: now also U14.6; no longer U14.6
- net at U25.3 (Q): now also U14.5; no longer U14.5
- new net: U1.117 (IO_L64P_SCP5_0), U14.1, U14.3

Commit message: cbmio 1.1a draft
Parts:
- R47, R48: footprint Resistor_SMD:R_0805_2012Metric_Pad1.20x1.40mm_HandSolder -> Resistor_SMD:R_0603_1608Metric_Pad0.98x0.95mm_HandSolder
Changed lines of the file:
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@@
 			)
 		)
-		(property "Footprint" "Resistor_SMD:R_0805_2012Metric_Pad1.20x1.40mm_HandSolder"
+		(property "Footprint" "Resistor_SMD:R_0603_1608Metric_Pad0.98x0.95mm_HandSolder"
 			(at 41.91 327.66 0)
 			(hide yes)
@@
 			)
 		)
-		(property "Footprint" "Resistor_SMD:R_0805_2012Metric_Pad1.20x1.40mm_HandSolder"
+		(property "Footprint" "Resistor_SMD:R_0603_1608Metric_Pad0.98x0.95mm_HandSolder"
 			(at 46.99 166.37 0)
 			(hide yes)

Commit message: fix DIN-6 connector BOM
Parts:
- J1: LCSC (none) -> C53056242
Changed lines of the file:
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@@
+			)
+		)
+		(property "LCSC" "C53056242"
+			(at 66.04 39.37 0)
+			(hide yes)
+			(show_name no)
+			(do_not_autoplace no)
+			(effects
+				(font
+					(size 1.27 1.27)
+				)
 			)
 		)
