File: Board/csa_petio_v1.kicad_pcb (KiCad board)
At the start: 6 copper layers, 160 x 100 mm, 61 parts, among them IC16 74LVC8T245SO24, IC3 7400N, J1 DIN-6, J11 Conn_01x09, J12 Conn_01x09, J14 Extended_PET_keyboard_connect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, J2 Conn_01x23, P2 IEEE488FLATCABLE, P3 PETUSERPORT, P4 CSABUS, P5 CBMTAPE, P6 CBMTAPE, U1 XC6SLX9-TQG144, U10 74LS06, U11 SN74LVC245APW, U12 4051, U13 4051, U14 74LVC1G04, U15 ADM560, U2 SN74LVC245APW, U3 SN74LVC245APW, U4 SN75160BDW, U5 SN75161BDW, U6 LSF0204Q, U7 LSF0204Q, U8 LSF0204Q, U9 LSF0204Q, X3 M09HPS

Commit message: schematics 1st full rev
Parts:
- removed C1: 100n, Capacitor_SMD:C_0805_2012Metric
- removed IC3: 7400N, csa_petio_v1:DIL14
- removed JP11, JP4: JP1E, csa_petio_v1:JP1
- removed P3: PETUSERPORT, csa_petio_v1:FLAT24
- removed P6: CBMTAPE, csa_petio_v1:JP6
- removed U$2: TASTER, csa_petio_v1:TASTER
- added C10: 100n, Capacitor_SMD:C_0805_2012Metric, F.Cu at (88.3, 36.9)
- added C15: 100n, Capacitor_SMD:C_0805_2012Metric, F.Cu at (88.3, 39.9)
- added C16: 100n, Capacitor_SMD:C_0805_2012Metric, F.Cu at (88.3, 42.9)
- added C17: 100n, Capacitor_SMD:C_0805_2012Metric, F.Cu at (88.3, 45.9)
- added C18: 100n, Capacitor_SMD:C_0805_2012Metric, F.Cu at (92.7, 33.9)
- added C19: 100n, Capacitor_SMD:C_0805_2012Metric, F.Cu at (92.7, 36.9)
- added C20: 100n, Capacitor_SMD:C_0805_2012Metric, F.Cu at (92.7, 39.9)
- added C21: 100n, Capacitor_SMD:C_0805_2012Metric, F.Cu at (92.7, 42.9)
- added C23: 100n, Capacitor_SMD:C_0805_2012Metric, F.Cu at (92.7, 45.9)
- added C24: 100n, Capacitor_SMD:C_0805_2012Metric, F.Cu at (97.2, 33.9)
- added C25: 100n, Capacitor_SMD:C_0805_2012Metric, F.Cu at (97.2, 36.9)
- added C26: 100n, Capacitor_SMD:C_0805_2012Metric, F.Cu at (97.2, 39.9)
- added C9: 100n, Capacitor_SMD:C_0805_2012Metric, F.Cu at (88.3, 33.9)
- added P1: PETUSERPORT, csa_petio_v1:FLAT24, F.Cu at (166.6, 130.1)
- added R10: 1k, Resistor_SMD:R_0603_1608Metric_Pad0.98x0.95mm_HandSolder, F.Cu at (236.5, 97.6)
- added R9: 1k, Resistor_SMD:R_0603_1608Metric_Pad0.98x0.95mm_HandSolder, F.Cu at (236.5, 95.1)
- added RN2: 10k, Resistor_THT:R_Array_SIP9, F.Cu at (182.9, 75.4)
- added RN3: 10k, Resistor_THT:R_Array_SIP9, F.Cu at (186.7, 112.0)
- added RN4: 10k, Resistor_THT:R_Array_SIP9, F.Cu at (177.3, 139.2)
- added RN5: 10k, Resistor_THT:R_Array_SIP9, F.Cu at (173.2, 139.2)
- added U16: LSF0204Q, Package_SO:TSSOP-14_4.4x5mm_P0.65mm, F.Cu at (141.0, 122.1)
- added U17: LSF0204Q, Package_SO:TSSOP-14_4.4x5mm_P0.65mm, F.Cu at (141.7, 146.9)
- added U18: LSF0204Q, Package_SO:TSSOP-14_4.4x5mm_P0.65mm, F.Cu at (142.1, 140.2)
- added U19: LSF0204Q, Package_SO:TSSOP-14_4.4x5mm_P0.65mm, F.Cu at (141.5, 132.3)
- added U20: ~, Connector_IDC:IDC-Header_2x13_P2.54mm_Vertical, F.Cu at (153.5, 116.4)
- added U21: 74LVC1G125, Package_TO_SOT_SMD:SOT-353_SC-70-5, F.Cu at (101.5, 34.4)
- added U22: 74LVC1G125, Package_TO_SOT_SMD:SOT-353_SC-70-5, F.Cu at (101.5, 38.3)
- added U23: 74LVC1G00, Package_TO_SOT_SMD:SOT-353_SC-70-5_Handsoldering, F.Cu at (174.2, 149.2)
- moved JP1 107.3 mm to (106.2, 112.5)
- moved R5 105.2 mm to (106.4, 137.4)
- moved C2 102.9 mm to (95.1, 125.4)
- moved C3 100.7 mm to (90.9, 125.2)
- moved C5 95.8 mm to (104.4, 123.0)
- moved C4 95.8 mm to (104.4, 120.0)
- moved C6 95.8 mm to (104.4, 126.0)
- moved UX18 95.0 mm to (126.0, 121.7)
- moved UX17 93.9 mm to (89.7, 133.9)
- moved C8 91.8 mm to (86.1, 125.0)
- moved C7 91.8 mm to (86.1, 122.0)
- moved UX16 87.4 mm to (100.8, 133.3)
- moved P5 77.5 mm to (195.0, 110.5), turned to 90 degrees
- moved UX7 74.1 mm to (196.9, 77.5)
- moved J12 63.4 mm to (85.6, 148.2), turned to 90 degrees
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Connections:
- net Net-(U4-D1) renamed UD1
- net Net-(U4-D2) renamed UD2
- net Net-(U4-D3) renamed UD3
- net Net-(U4-D4) renamed UD4
- net Net-(U4-D5) renamed UD5
- net Net-(U4-D6) renamed UD6
- net Net-(U4-D7) renamed UD7
- net Net-(U4-D8) renamed UD8
- IC16 pad 22: /IOSEL -> /BE
- P5 pad 3: /C1MTR -> C1MTR
- P5 pad 4: /C1RD -> C1RD
- P5 pad 5: /CWR -> CWR
- P5 pad 6: /C1SW -> C1SW
- U1 pad 111: unconnected-(U1A-IO_L66N_SCP0_0-Pad111) -> UP7
- U1 pad 112: unconnected-(U1A-IO_L66P_SCP1_0-Pad112) -> UP6
- U1 pad 134: CLKOUT -> Net-(U11-B1)
- U1 pad 137: Net-(U11-B8) -> UP11
- U1 pad 138: Net-(U11-B7) -> UP10
- U1 pad 139: Net-(U11-B6) -> UP9
- U1 pad 140: Net-(U11-B5) -> UP8
- U1 pad 144: Net-(U11-B1) -> CLKOUT
- U1 pad 35: unconnected-(U1B-IO_L1P_3-Pad35) -> /BE
- U1 pad 58: unconnected-(U1B-IO_L14P_D11_2-Pad58) -> C1SW
- U1 pad 59: unconnected-(U1B-IO_L13N_D10_2-Pad59) -> C1RD
- U1 pad 60: unconnected-(U1B-IO_L13P_M1_2-Pad60) -> CWR
- U1 pad 61: unconnected-(U1B-IO_L12N_D2_MISO3_2-Pad61) -> C1MTR
- U1 pad 62: unconnected-(U1B-IO_L12P_D1_MISO2_2-Pad62) -> UP12
- U1 pad 69: unconnected-(U1B-IO_L1N_M0_CMPMISO_2-Pad69) -> UP13
- U1 pad 74: unconnected-(U1A-IO_L74N_DOUT_BUSY_1-Pad74) -> UP5
- U1 pad 75: unconnected-(U1A-IO_L74P_AWAKE_1-Pad75) -> UP4
- U1 pad 78: unconnected-(U1A-IO_L47N_1-Pad78) -> UP3
- U1 pad 79: unconnected-(U1A-IO_L47P_1-Pad79) -> UP2
- U1 pad 80: unconnected-(U1A-IO_L46N_1-Pad80) -> UP1
- U1 pad 81: unconnected-(U1A-IO_L46P_1-Pad81) -> UP0
- U1 pad 82: unconnected-(U1A-IO_L45N_1-Pad82) -> Net-(U1A-IO_L45N_1)
- U10 pad 11: unconnected-(U10-Pad11) -> Net-(R10-Pad1)
- U11 pad 11: Net-(U11-B8) -> unconnected-(U11-B8-Pad11)
- U11 pad 12: Net-(U11-B7) -> unconnected-(U11-B7-Pad12)
- U11 pad 13: Net-(U11-B6) -> unconnected-(U11-B6-Pad13)
- U11 pad 14: Net-(U11-B5) -> unconnected-(U11-B5-Pad14)
- U11 pad 6: unconnected-(U11-A5-Pad6) -> Net-(U11-A5)
- U11 pad 7: unconnected-(U11-A6-Pad7) -> Net-(U11-A5)
- U11 pad 8: unconnected-(U11-A7-Pad8) -> Net-(U11-A5)
- U11 pad 9: unconnected-(U11-A8-Pad9) -> Net-(U11-A5)
- U4 pad 1: Net-(U1A-IO_L43N_GCLK4_1) -> Net-(U1A-IO_L45P_1)
- U5 pad 1: Net-(U1A-IO_L43N_GCLK4_1) -> Net-(U1A-IO_L45P_1)
- U5 pad 11: Net-(U1A-IO_L45P_1) -> Net-(U1A-IO_L45N_1)
- U6 pad 1: unconnected-(U6-VRefA-Pad1) -> GND
- U6 pad 14: unconnected-(U6-VRefB-Pad14) -> GND
- U6 pad 2: unconnected-(U6-A1-Pad2) -> Net-(U1A-IO_L1P_1)
- U6 pad 3: Net-(U1A-IO_L1P_1) -> Net-(U1A-IO_L1N_VREF_1)
- U6 pad 4: Net-(U1A-IO_L1N_VREF_1) -> Net-(U1A-IO_L32P_1)
- U6 pad 5: Net-(U1A-IO_L32P_1) -> Net-(U1A-IO_L32N_1)
- U7 pad 1: unconnected-(U7-VRefA-Pad1) -> GND
- U7 pad 14: unconnected-(U7-VRefB-Pad14) -> GND
- U7 pad 2: Net-(U1A-IO_L32N_1) -> Net-(U1A-IO_L33P_1)
- U7 pad 3: Net-(U1A-IO_L33P_1) -> Net-(U1A-IO_L33N_1)
- U7 pad 4: Net-(U1A-IO_L33N_1) -> Net-(U1A-IO_L34P_1)
- U7 pad 5: Net-(U1A-IO_L34P_1) -> Net-(U1A-IO_L34N_1)
- U8 pad 1: unconnected-(U8-VRefA-Pad1) -> GND
- U8 pad 14: unconnected-(U8-VRefB-Pad14) -> GND
- U8 pad 2: Net-(U1A-IO_L34N_1) -> Net-(U1A-IO_L40P_GCLK11_1)
- U8 pad 3: Net-(U1A-IO_L40P_GCLK11_1) -> Net-(U1A-IO_L40N_GCLK10_1)
- U8 pad 4: Net-(U1A-IO_L40N_GCLK10_1) -> Net-(U1A-IO_L41P_GCLK9_IRDY1_1)
- U8 pad 5: Net-(U1A-IO_L41P_GCLK9_IRDY1_1) -> Net-(U1A-IO_L41N_GCLK8_1)
- U9 pad 1: unconnected-(U9-VRefA-Pad1) -> GND
- U9 pad 14: unconnected-(U9-VRefB-Pad14) -> GND
- U9 pad 2: Net-(U1A-IO_L41N_GCLK8_1) -> Net-(U1A-IO_L42P_GCLK7_1)
- U9 pad 3: Net-(U1A-IO_L42P_GCLK7_1) -> Net-(U1A-IO_L42N_GCLK6_TRDY1_1)
- U9 pad 4: Net-(U1A-IO_L42N_GCLK6_TRDY1_1) -> Net-(U1A-IO_L43P_GCLK5_1)
- U9 pad 5: Net-(U1A-IO_L43P_GCLK5_1) -> Net-(U1A-IO_L43N_GCLK4_1)
Other:
- board text removed: "C64"
- board text removed: "Ext Pwr"
- board text removed: "GND VCC"
- board text removed: "PET"

Commit message: full connect, starting on prod
Parts:
- added C1: 100n, Capacitor_SMD:C_0805_2012Metric, F.Cu at (122.1, 84.8)
- added C22: 100n, Capacitor_SMD:C_0805_2012Metric, F.Cu at (138.4, 102.6)
- added C27: 100n, Capacitor_SMD:C_0805_2012Metric, F.Cu at (105.7, 102.4)
- added C28: 100n, Capacitor_SMD:C_0805_2012Metric, F.Cu at (120.9, 117.9)
- added C29: 100n, Capacitor_SMD:C_0805_2012Metric, F.Cu at (105.7, 93.7)
- added C30: 100n, Capacitor_SMD:C_0805_2012Metric, F.Cu at (105.7, 100.3)
- added C31: 100n, Capacitor_SMD:C_0805_2012Metric, F.Cu at (105.7, 110.5)
- added C32: 100n, Capacitor_SMD:C_0805_2012Metric, F.Cu at (115.8, 84.8)
- added C33: 100n, Capacitor_SMD:C_0805_2012Metric, F.Cu at (125.5, 84.6)
- added C34: 100n, Capacitor_SMD:C_0805_2012Metric, F.Cu at (138.4, 94.5)
- added C35: 100n, Capacitor_SMD:C_0805_2012Metric, F.Cu at (119.6, 84.8)
- added C36: 100n, Capacitor_SMD:C_0805_2012Metric, F.Cu at (138.4, 100.6)
- added C37: 100n, Capacitor_SMD:C_0805_2012Metric, F.Cu at (138.4, 108.7)
- added C38: 100n, Capacitor_SMD:C_0805_2012Metric, F.Cu at (115.8, 117.9)
- added C39: 100n, Capacitor_SMD:C_0805_2012Metric, F.Cu at (123.4, 117.9)
- added C40: 100n, Capacitor_SMD:C_0805_2012Metric, F.Cu at (127.0, 117.9)
- added RN6: 4k7, Resistor_THT:R_Array_SIP5, F.Cu at (202.4, 91.4)
- IC16: footprint Package_SO:SO-24_5.3x15mm_P1.27mm -> Package_SO:TSSOP-24_6.1x7.8mm_P0.65mm
- P1, P2: footprint csa_petio_v1:FLAT24 -> csa_petio_v1:FLAT24_IDC
- moved JP18 147.1 mm to (137.1, 59.4)
- moved JP22 147.1 mm to (141.7, 59.4)
- moved R9 127.4 mm to (109.7, 82.3), turned to -90 degrees
- moved R10 126.8 mm to (112.5, 71.4), turned to 180 degrees
- moved UX7 110.4 mm to (87.1, 65.5), turned to 90 degrees
- moved C18 109.4 mm to (122.4, 139.2), turned to 180 degrees
- moved C19 105.8 mm to (129.3, 136.1), turned to 180 degrees
- moved R1 97.2 mm to (100.1, 125.2), turned to -90 degrees
- moved R2 96.7 mm to (121.9, 135.9), turned to 180 degrees
- moved C25 95.2 mm to (173.0, 94.5), turned to 180 degrees
- moved C24 90.1 mm to (89.9, 123.7)
- moved R4 89.7 mm to (131.3, 118.1), turned to 90 degrees
- moved P9 89.6 mm to (205.5, 113.5)
- moved U21 83.9 mm to (104.6, 118.2)
- moved U22 83.9 mm to (104.6, 122.2)
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Connections:
- BEEP1 pad 2: V12 -> GND
- C10 pad 2: V12 -> GND
- C13 pad 2: V12 -> V33
- C14 pad 1: V12 -> GND
- C15 pad 2: V12 -> GND
- C16 pad 2: V12 -> GND
- C17 pad 2: V12 -> GND
- C18 pad 2: V12 -> GND
- C19 pad 2: V12 -> GND
- C2 pad 1: GND -> VCC
- C2 pad 2: V12 -> GND
- C20 pad 2: V12 -> GND
- C21 pad 2: V12 -> GND
- C23 pad 1: GND -> VCC
- C23 pad 2: V12 -> GND
- C24 pad 1: GND -> VCC
- C24 pad 2: V12 -> GND
- C25 pad 1: GND -> VCC
- C25 pad 2: V12 -> GND
- C26 pad 1: GND -> VCC
- C26 pad 2: V12 -> GND
- C3 pad 2: V12 -> GND
- C4 pad 2: V12 -> GND
- C5 pad 1: GND -> VCC
- C5 pad 2: V12 -> GND
- C6 pad 2: V12 -> GND
- C7 pad 2: V12 -> GND
- C8 pad 1: GND -> VCC
- C8 pad 2: V12 -> GND
- C9 pad 2: V12 -> GND
- IC16 pad 11: V12 -> GND
- IC16 pad 12: V12 -> GND
- IC16 pad 13: V12 -> GND
- IC16 pad 23: V12 -> VCC
- IC16 pad 24: V12 -> VCC
- J1 pad 2: V12 -> GND
- J11 pad 1: V12 -> GND
- J12 pad 1: V12 -> GND
- J14 pad 1: V12 -> GND
- J14 pad 21: V12 -> GND
- J14 pad 26: GND -> VCC
- J14 pad 27: GND -> V33
- JP1 pad 2: V12 -> GND
- P1 pad 1: V12 -> GND
- P1 pad 12: V12 -> GND
- P1 pad 2: GND -> VCC
- P1 pad A: V12 -> GND
- P1 pad N: V12 -> GND
- P2 pad 12: V12 -> GND
- P2 pad E: V12 -> GND
- P2 pad F: V12 -> GND
- P2 pad H: V12 -> GND
- P2 pad J: V12 -> GND
- P2 pad K: V12 -> GND
- P2 pad L: V12 -> GND
- P2 pad M: V12 -> GND
- P2 pad N: V12 -> GND
- P4 pad A1: V12 -> GND
- P4 pad A28: V12 -> GND
- P4 pad A29: V12 -> GND
- P4 pad A30: V12 -> GND
- P4 pad A31: V12 -> GND
- P4 pad A32: V12 -> GND
- P4 pad C1: V12 -> GND
- P4 pad C2: V12 -> VCC
- P4 pad C26: V12 -> Net-(P4-PHI2)
- P4 pad C3: V12 -> VCC
- P4 pad C32: V12 -> GND
- P5 pad 1: V12 -> GND
- P5 pad 2: GND -> VCC
- P9 pad 1: GND -> VCC
- P9 pad 2: V12 -> GND
- R10 pad 2: V12 -> GND
- R3 pad 2: GND -> VCC
- R5 pad 1: GND -> VCC
- R8 pad 2: V12 -> GND
- R9 pad 2: V12 -> GND
- RN1 pad 1: GND -> V33
- RN2 pad 1: GND -> VCC
- RN3 pad 1: GND -> VCC
- RN4 pad 1: GND -> VCC
- RN5 pad 1: unconnected-(RN5-common-Pad1) -> VCC
- U1 pad 103: GND -> V33
- U1 pad 108: V12 -> GND
- U1 pad 113: V12 -> GND
- U1 pad 122: GND -> V33
- U1 pad 125: GND -> V33
- U1 pad 13: V12 -> GND
- U1 pad 130: V12 -> GND
- U1 pad 135: GND -> V33
- U1 pad 136: V12 -> GND
- U1 pad 18: V12 -> V33
- U1 pad 25: V12 -> GND
- U1 pad 3: V12 -> GND
- U1 pad 31: V12 -> V33
- U1 pad 39: /IO1/LDCD -> /IO1/LCTS
- U1 pad 4: V12 -> V33
- U1 pad 40: /IO1/LCTS -> /IO1/LTX
- U1 pad 41: /IO1/LDSR -> /IO1/LRX
- U1 pad 42: V12 -> V33
- U1 pad 43: /IO1/LRI -> /IO1/LRTS
- U1 pad 44: /IO1/LRX -> /IO1/LDSR
- U1 pad 45: /IO1/LTX -> /IO1/LDTR
- U1 pad 46: /IO1/LDTR -> /IO1/LDCD
- U1 pad 47: /IO1/LRTS -> /IO1/LRI
- U1 pad 49: V12 -> GND
- U1 pad 54: V12 -> GND
- U1 pad 63: V12 -> V33
- U1 pad 68: V12 -> GND
- U1 pad 76: GND -> V33
- U1 pad 77: V12 -> GND
- U1 pad 86: GND -> V33
- U1 pad 91: V12 -> GND
- U1 pad 96: V12 -> GND
- U10 pad 14: GND -> VCC
- U10 pad 7: V12 -> GND
- U11 pad 1: GND -> V33
- U11 pad 10: V12 -> GND
- U11 pad 20: GND -> V33
- U12 pad 16: GND -> V33
- U12 pad 3: V12 -> GND
- U12 pad 7: V12 -> GND
- U12 pad 8: V12 -> GND
- U13 pad 16: GND -> V33
- U13 pad 3: V12 -> GND
- U13 pad 7: V12 -> GND
- U13 pad 8: V12 -> GND
- U14 pad 3: V12 -> GND
- U14 pad 5: GND -> V33
- U15 pad 10: V12 -> GND
- U15 pad 11: V12 -> V33
- U15 pad 24: V12 -> V33
- U15 pad 25: V12 -> V33
- U16 pad 14: GND -> VCC
- U16 pad 7: V12 -> GND
- U17 pad 14: GND -> VCC
- U17 pad 7: V12 -> GND
- U18 pad 14: GND -> VCC
- U18 pad 7: V12 -> GND
- U19 pad 14: GND -> VCC
- U19 pad 7: V12 -> GND
- U2 pad 10: V12 -> GND
- U2 pad 19: V12 -> GND
- U2 pad 2: V12 -> Net-(P4-PHI2)
- U20 pad 1: V12 -> GND
- U20 pad 24: GND -> VCC
- U20 pad 3: V12 -> GND
- U21 pad 2: V12 -> GND
- U21 pad 3: V12 -> GND
- U22 pad 2: V12 -> GND
- U22 pad 3: V12 -> GND
- U23 pad 3: V12 -> GND
- U23 pad 5: GND -> VCC
- U3 pad 10: V12 -> GND
- U3 pad 19: V12 -> GND
- U4 pad 10: V12 -> GND
- U4 pad 20: GND -> VCC
- U5 pad 10: V12 -> GND
- U5 pad 20: GND -> VCC
- U6 pad 1: GND -> V33
- U6 pad 14: GND -> VCC
- U6 pad 7: V12 -> GND
- U7 pad 1: GND -> V33
- U7 pad 14: GND -> VCC
- U7 pad 7: V12 -> GND
- U8 pad 1: GND -> V33
- U8 pad 14: GND -> VCC
- U8 pad 7: V12 -> GND
- U9 pad 1: GND -> V33
- U9 pad 14: GND -> VCC
- U9 pad 7: V12 -> GND
- UX16 pad 3: GND -> VCC
- UX16 pad 4: GND -> VCC
- UX16 pad 7: V12 -> GND
- UX16 pad 8: V12 -> GND
- UX17 pad 1: V12 -> GND
- UX17 pad 3: GND -> VCC
- UX18 pad 4: V12 -> GND
- X3 pad 5: V12 -> GND
Routing:
- net GND: track 0.00 -> 874.9 mm, vias 0 -> 74
- net V33: track 0.00 -> 866.4 mm, vias 0 -> 79
- net VCC: track 0.00 -> 552.0 mm, vias 0 -> 22
- net /BIRQ: track 0.00 -> 274.0 mm, vias 0 -> 10
- net /RES: track 0.00 -> 229.9 mm, vias 0 -> 16
- net /BRES: track 0.00 -> 189.5 mm, vias 0 -> 3
- net CLKOUT: track 0.00 -> 188.1 mm, vias 0 -> 7
- net /IO2/SLOWCLK: track 0.00 -> 161.4 mm, vias 0 -> 6
- net V12: track 0.00 -> 161.4 mm, vias 0 -> 7
- net /IO2/DATA: track 0.00 -> 161.1 mm, vias 0 -> 6
- net /IO2/SATN: track 0.00 -> 151.9 mm, vias 0 -> 4
- net /IO2/FASTCLK: track 0.00 -> 143.7 mm, vias 0 -> 5
- net SPI_CLK: track 0.00 -> 134.7 mm, vias 0 -> 4
- net Net-(P9-MISO): track 0.00 -> 131.0 mm, vias 0 -> 5
- net /IO1/DTR: track 0.00 -> 129.7 mm, vias 0 -> 2
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Other:
- copper layers 6 -> 2
- board text added: "CBMUSER"

Commit message: fix version on PCB
Other:
- board text added: "CSA-CBMIO-V1.0A"
- board text removed: "CSA-PETIO-V1.3B"

Commit message: prod files
Parts:
- R5: value 10k -> 4k7
Routing:
- net VCC: track 552.0 -> 754.8 mm, vias 22 -> 33
- net GND: track 874.9 -> 943.6 mm, vias 74 -> 82
- net V33: track 866.4 -> 885.9 mm, vias 79 -> 81
- net V12: track 161.4 -> 168.9 mm, vias 7 -> 9
- net KSEL0: track 102.8 -> 104.9 mm
- net KSEL2: track 102.7 -> 101.6 mm
- net Net-(P1-PA4): track 87.7 -> 86.8 mm
- net /BIRQ: track 274.0 -> 273.2 mm
- net Net-(J2-Pin_1): track 116.3 -> 117.1 mm
- net KSEL1: track 102.6 -> 101.8 mm
- net /IO2/DATA: track 161.1 -> 160.4 mm
- net Net-(J2-Pin_2): track 121.6 -> 122.1 mm
Other:
- board text added: "(U)PETKBD"
- board text added: "1 Serial 2"
- board text added: "CBMKBD"
- board text added: "CBMTAPE1"
- board text added: "CTS TX RX RTS DSR DTR CD RI"
- board text added: "FPGAPROG"
- board text added: "IEC Bus"
- board text added: "IEEE488"
- board text added: "PETUSER"
- board text added: "PROG"
- board text added: "SPI-10-5V"
- board text added: "Serial 1 / RS232"
