File: Board/csa_petio_v1.kicad_pcb (KiCad board)
At the start: 2 copper layers, 160 x 100 mm, 99 parts, among them IC16 74LVC8T245SO24, J1 DIN-6, J11 Conn_01x09, J12 Conn_01x09, J14 Extended_PET_keyboard_connect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, J2 Conn_01x23, P1 PETUSERPORT, P2 IEEE488FLATCABLE, P4 CSABUS, P5 CBMTAPE, U1 XC6SLX9-TQG144, U10 74LS06, U11 SN74LVC245APW, U12 4051, U13 4051, U14 74LVC1G04, U15 ADM560, U16 LSF0204Q, U17 LSF0204Q, U18 LSF0204Q, U19 LSF0204Q, U2 SN74LVC245APW, U21 74LVC1G125, U22 74LVC1G125, U23 74LVC1G00, U3 SN74LVC245APW, U4 SN75160BDW, U5 SN75161BDW, U6 LSF0204Q, U7 LSF0204Q, U8 LSF0204Q, U9 LSF0204Q, X3 M09HPS

Commit message: 1st working as 1.0B
Parts:
- R5: value 4k7 -> 10k
Connections:
- U1 pad 1: PHI2 -> /IRQ
- U1 pad 23: /IRQ -> PHI2
- UX7 pad 10: (no net) -> GND
- UX7 pad 2: (no net) -> GND
- UX7 pad 4: (no net) -> V33
Routing:
- net V33: track 885.9 -> 905.8 mm
- net /IRQ: track 67.4 -> 56.0 mm
- net PHI2: track 20.1 -> 31.2 mm, vias 0 -> 2
- net GND: track 943.6 -> 948.8 mm
Other:
- board text added: "CSA-CBMIO-V1.0B"
- board text removed: "CSA-CBMIO-V1.0A"
