File: Board/fpga.kicad_sch (KiCad schematic)
At the start: 48 parts, among them U1 XC6SLX9-TQG144, U21 74LVC1G125, U22 74LVC1G125

Commit message: start working on 1.0b
Other:
- note added: "CSA-CBMIO-V1.0B"
- note removed: "CSA-CBMIO-V1.0A"
Changed lines of the file:
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@@
 	(generator_version "9.0")
 	(paper "A4")
-	(text "CSA-CBMIO-V1.0A"
+	(text "CSA-CBMIO-V1.0B"
 		(exclude_from_sim no)
 		(at 206.756 172.72 0)
