File: Board/fpga.kicad_sch (KiCad schematic)
At the start: 48 parts, among them U1 XC6SLX9-TQG144, U21 74LVC1G125, U22 74LVC1G125

Commit message: added comments and TODOs on schem
Parts:
- added unit 2 of UX7
- added unit 3 of UX7
Connections:
- net GND: now also UX7.10 (P$1), UX7.2 (GND); no longer UX7.10 (P$1), UX7.2 (GND)
- net V33: now also UX7.4 (VCC); no longer UX7.4 (VCC)
Changed lines of the file:
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@@
 		)
 		(instances
-			(project ""
+			(project "csa_petio_v1"
 				(path "/e52c695d-6540-4a56-9880-06c7d9f215a5/68abe788-b880-40e7-9e78-97f20b071325"
 					(reference "U21")
@@
 		)
 		(instances
-			(project ""
+			(project "csa_petio_v1"
 				(path "/e52c695d-6540-4a56-9880-06c7d9f215a5/68abe788-b880-40e7-9e78-97f20b071325"
 					(reference "U1")
@@
 		)
 		(instances
-			(project ""
+			(project "csa_petio_v1"
 				(path "/e52c695d-6540-4a56-9880-06c7d9f215a5/68abe788-b880-40e7-9e78-97f20b071325"
 					(reference "R1")
@@
 		)
 		(instances
-			(project ""
+			(project "csa_petio_v1"
 				(path "/e52c695d-6540-4a56-9880-06c7d9f215a5/68abe788-b880-40e7-9e78-97f20b071325"
 					(reference "C4")

Commit message: add par ATNA, separate kbd cons, kbd serial input to get more I/O
Other:
- note added: "CSA-CBMIO-V1.1A"
- note removed: "CSA-CBMIO-V1.0B"
