File: Board/fpga.kicad_sch (KiCad schematic)
At the start: 48 parts, among them U1 XC6SLX9-TQG144, U21 74LVC1G125, U22 74LVC1G125

Commit message: schem draft done, layout work started
Parts:
- added C41: 100n, Capacitor_SMD:C_0805_2012Metric, symbol Device:C
Connections:
- net GND: now also C41.2
- net VCC: now also C41.1
Other:
- note added: "CSA-CBMIO-V1.1A-20260824"
- note removed: "CSA-CBMIO-V1.0B-20260321"
Changed lines of the file:
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@@
 		)
 	)
-	(text "CSA-CBMIO-V1.0B-20260321"
+	(text "CSA-CBMIO-V1.1A-20260824"
 		(exclude_from_sim no)
 		(at 209.296 186.436 0)
@@
 	)
 	(junction
+		(at 201.93 158.75)
+		(diameter 0)
+		(color 0 0 0 0)
+	)
+	(junction
 		(at 248.92 143.51)
 		(diameter 0)
@@
 	)
 	(junction
+		(at 201.93 151.13)
+		(diameter 0)
+		(color 0 0 0 0)
+	)
+	(junction
 		(at 110.49 171.45)
 		(diameter 0)
@@
 	(wire
 		(pts
+			(xy 201.93 151.13) (xy 213.36 151.13)
+		)
+		(stroke
+			(width 0)
+			(type default)
+		)
+	)
+	(wire
+		(pts
 			(xy 194.31 74.93) (xy 196.85 74.93)
 		)
@@
 	(wire
 		(pts
+			(xy 201.93 158.75) (xy 213.36 158.75)
+		)
+		(stroke
+			(width 0)
+			(type default)
+		)
+	)
+	(wire
+		(pts
 			(xy 110.49 116.84) (xy 113.03 116.84)
 		)
@@
 					(unit 1)
 				)
+			)
+		)
+	)
+	(symbol
+		(lib_id "Device:C")
+		(at 213.36 154.94 0)
+		(unit 1)
+		(body_style 1)
+		(exclude_from_sim no)
+		(in_bom yes)
+		(on_board yes)
+		(in_pos_files yes)
+		(dnp no)
+		(fields_autoplaced yes)
+		(property "Reference" "C41"
+			(at 217.17 153.6699 0)
+			(show_name no)
+			(do_not_autoplace no)
+			(effects
+				(font
+					(size 1.27 1.27)
+				)
+				(justify left)
+			)
+		)
+		(property "Value" "100n"
+			(at 217.17 156.2099 0)
+			(show_name no)
+			(do_not_autoplace no)
+			(effects
+				(font
+					(size 1.27 1.27)
+				)
+				(justify left)
+			)
+		)
+		(property "Footprint" "Capacitor_SMD:C_0805_2012Metric"
+			(at 214.3252 158.75 0)
+			(hide yes)
+			(show_name no)
+			(do_not_autoplace no)
+			(effects
+				(font
+					(size 1.27 1.27)
+				)
+			)
+		)
+		(property "Datasheet" ""
+			(at 213.36 154.94 0)
+			(hide yes)
+			(show_name no)
+			(do_not_autoplace no)
+			(effects
+				(font
+					(size 1.27 1.27)
+				)
+			)
+		)
+		(property "Description" "Unpolarized capacitor"
+			(at 213.36 154.94 0)
+			(hide yes)
+			(show_name no)
+			(do_not_autoplace no)
+			(effects
+				(font
+					(size 1.27 1.27)
+				)
+			)
+		)
+		(pin "2"
+		)
+		(pin "1"
+		)
+		(instances
+			(project "csa_petio_v1"
+				(path "/e52c695d-6540-4a56-9880-06c7d9f215a5/68abe788-b880-40e7-9e78-97f20b071325"
+					(reference "C41")
+					(unit 1)
+				)
