File: Board/io1.kicad_sch (KiCad schematic)
At the start: 13 parts, among them J11 Conn_01x09, J12 Conn_01x09, P5 CBMTAPE, U1 XC6SLX9-TQG144, U15 ADM560, X3 M09HPS

Commit message: start working on 1.0b
Other:
- note added: "CSA-CBMIO-V1.0B"
- note removed: "CSA-CBMIO-V1.0A"
Changed lines of the file:
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@@
 		)
 	)
-	(text "CSA-CBMIO-V1.0A"
+	(text "CSA-CBMIO-V1.0B"
 		(exclude_from_sim no)
 		(at 331.47 261.112 0)
