File: Board/bus.kicad_sch (KiCad schematic)
At the start: 5 parts, among them IC16 74LVC8T245SO24, P4 CSABUS, U10 74LS06, U2 SN74LVC245APW, U3 SN74LVC245APW

Commit message: start working on 1.0b
Parts:
- IC16: footprint Package_SO:TSSOP-24_6.1x7.8mm_P0.65mm -> Package_SO:TSSOP-24_4.4x7.8mm_P0.65mm
Other:
- note added: "1.0B: - fix 74lvc8t245 footprint"
- note added: "CSA-CBMIO-V1.0B"
- note added: "CSA-CBMIO-V1.0B-20250825"
- note added: "Notes: - Note that the /OE (and DIR) inputs on the 8T245 reference VCCA, and are CMOS, so driving from 3.3V does not reach 3.5 Vi_hi_min; therefore bus is on B side"
- note removed: "CSA-CBMIO-V1.0A"
- note removed: "CSA-CBMIO-V1.0A-20250815"
- note removed: "Notes: - Note that the /OE (and DIR) outputs reference VCCA, and are CMOS, so driving from 3.3V does not reach 3.5 Vi_hi_min"
Changed lines of the file:
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@@
 	(generator_version "9.0")
 	(paper "A4")
-	(text "Notes:\n- Note that the /OE (and DIR) outputs reference VCCA, and are CMOS, so \n  driving from 3.3V does not reach 3.5 Vi_hi_min"
+	(text "Notes:\n- Note that the /OE (and DIR) inputs on the 8T245\n  reference VCCA, and are CMOS, so driving from 3.3V \n  does not reach 3.5 Vi_hi_min; therefore bus is on\n  B side"
 		(exclude_from_sim no)
 		(at 191.008 30.734 0)
 		(effects
 			(font
-				(size 1.27 1.27)
-			)
-			(justify left)
-		)
-	)
-	(text "CSA-CBMIO-V1.0A"
+				(size 2 2)
+			)
+			(justify left)
+		)
+	)
+	(text "CSA-CBMIO-V1.0B"
 		(exclude_from_sim no)
 		(at 186.69 173.99 0)
@@
 		)
 	)
-	(text "CSA-CBMIO-V1.0A-20250815"
+	(text "CSA-CBMIO-V1.0B-20250825"
 		(exclude_from_sim no)
 		(at 209.042 185.674 0)
@@
 			)
 			(justify left bottom)
+		)
+	)
+	(text "1.0B:\n- fix 74lvc8t245 footprint"
+		(exclude_from_sim no)
+		(at 198.12 152.4 0)
+		(effects
+			(font
+				(size 2 2)
+			)
+			(justify left)
 		)
 	)
@@
 			)
 		)
-		(property "Footprint" "Package_SO:TSSOP-24_6.1x7.8mm_P0.65mm"
+		(property "Footprint" "Package_SO:TSSOP-24_4.4x7.8mm_P0.65mm"
 			(at 146.05 63.5 0)
 			(effects

Commit message: add par ATNA, separate kbd cons, kbd serial input to get more I/O
Connections:
- net /BNMI: now reaches P4.A23 (/NMI)
Other:
- note added: "CSA-CBMIO-V1.1A"
- note removed: "CSA-CBMIO-V1.0B"
