File: Board/csa_petio_v1.kicad_sch (KiCad schematic)
At the start: 0 parts

Commit message: schem draft done, layout work started
Other:
- note added: "CBM I/O Board with FPGA"
- note added: "CSA-CBMIO-V1.1A"
- note added: "This board implements the I/O for either a Commodore PET, a Commodore B-Series, or the Ulti-PET using a single FPGA. The I/O can be addressed/used via the CS/A Bus and the /IOSEL signal (if activated at the right address for the specific model)"
Changed lines of the file:
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@@
 	(generator_version "10.0")
 	(paper "User" 520.243 335.763)
-	(sheet
-		(at 129.54 44.45)
+	(text "CBM I/O Board with FPGA"
+		(exclude_from_sim no)
+		(at 72.39 49.53 0)
+		(effects
+			(font
+				(size 3.81 3.81)
+				(thickness 0.508)
+				(bold yes)
+			)
+		)
+	)
+	(text "CSA-CBMIO-V1.1A"
+		(exclude_from_sim no)
+		(at 414.02 302.26 0)
+		(effects
+			(font
+				(size 3.81 3.2385)
+			)
+			(justify left bottom)
+		)
+	)
+	(text "This board implements the I/O for either a Commodore PET, a \nCommodore B-Series, or the Ulti-PET using a single FPGA.\n\nThe I/O can be addressed/used via the CS/A Bus and the /IOSEL\nsignal (if activated at the right address for the specific\nmodel)"
+		(exclude_from_sim no)
+		(at 34.29 80.01 0)
+		(effects
+			(font
+				(size 2.54 2.54)
+				(thickness 0.254)
+				(bold yes)
+			)
+			(justify left)
+		)
+	)
+	(sheet
+		(at 130.81 297.18)
 		(size 15.24 8.89)
 		(exclude_from_sim no)
@@
 		)
 		(property "Sheetname" "IO1"
-			(at 129.54 43.7384 0)
+			(at 130.81 296.4684 0)
 			(show_name no)
 			(do_not_autoplace no)
@@
 		)
 		(property "Sheetfile" "io1.kicad_sch"
-			(at 129.54 53.9246 0)
+			(at 130.81 306.6546 0)
 			(show_name no)
 			(do_not_autoplace no)
@@
 	)
 	(sheet
-		(at 53.975 42.545)
+		(at 55.245 295.275)
 		(size 12.7 10.795)
 		(exclude_from_sim no)
@@
 		)
 		(property "Sheetname" "Bus"
-			(at 53.975 41.8334 0)
+			(at 55.245 294.5634 0)
 			(show_name no)
 			(do_not_autoplace no)
@@
 		)
 		(property "Sheetfile" "bus.kicad_sch"
-			(at 53.975 53.9246 0)
+			(at 55.245 306.6546 0)
 			(show_name no)
 			(do_not_autoplace no)
@@
 	)
 	(sheet
-		(at 92.71 43.815)
+		(at 93.98 296.545)
 		(size 12.7 11.43)
 		(exclude_from_sim no)
@@
 		)
 		(property "Sheetname" "FPGA"
-			(at 92.71 43.1034 0)
+			(at 93.98 295.8334 0)
 			(show_name no)
 			(do_not_autoplace no)
@@
 		)
 		(property "Sheetfile" "fpga.kicad_sch"
-			(at 92.71 55.8296 0)
+			(at 93.98 308.5596 0)
 			(show_name no)
 			(do_not_autoplace no)
@@
 	)
 	(sheet
-		(at 164.465 44.45)
+		(at 165.735 297.18)
 		(size 12.7 11.43)
 		(exclude_from_sim no)
@@
 		)
 		(property "Sheetname" "IO2"
-			(at 164.465 43.7384 0)
+			(at 165.735 296.4684 0)
 			(show_name no)
 			(do_not_autoplace no)
@@
 		)
 		(property "Sheetfile" "io2.kicad_sch"
-			(at 164.465 56.4646 0)
+			(at 165.735 309.1946 0)
 			(show_name no)
 			(do_not_autoplace no)
@@
 	)
 	(sheet
-		(at 199.39 41.91)
+		(at 200.66 294.64)
 		(size 12.7 10.795)
 		(exclude_from_sim no)
@@
 		)
 		(property "Sheetname" "Userport"
-			(at 199.39 41.1984 0)
+			(at 200.66 293.9284 0)
 			(show_name no)
 			(do_not_autoplace no)
@@
 		)
 		(property "Sheetfile" "userport.kicad_sch"
-			(at 199.39 53.2896 0)
-			(show_name no)
-			(do_not_autoplace no)
+			(at 200.66 306.0196 0)
+			(show_name no)
+			(do_not_autoplace no)
